Commit message: Testing new motion controller

File: pepper_robot/pepper_description/urdf/pepper1.0_generated_urdf/pepper_arms.xacro (robot description, xacro)
@@ -37,5 +37,6 @@
 		<parent link="LBicep"/>
 		<child link="LElbow"/>
-		<origin rpy="0 -0.157079 0" xyz="0.1812 0.015 0.00013"/>
+		<!-- <origin rpy="0 -0.157079 0" xyz="0.1812 0.015 0.00013"/> -->
+		<origin rpy="0 -0.0 0" xyz="0.1812 0.015 0.00013"/>
 		<axis xyz="1.0 0 0"/>
 		<limit effort="5.428" lower="-2.08567" upper="2.08567" velocity="7.33998"/>
@@ -125,5 +126,6 @@
 		<parent link="RBicep"/>
 		<child link="RElbow"/>
-		<origin rpy="0 -0.157079 0" xyz="0.1812 -0.015 0.00013"/>
+		<!-- <origin rpy="0 -0.157079 0" xyz="0.1812 -0.015 0.00013"/> -->
+		<origin rpy="0 -0.0 0" xyz="0.1812 -0.015 0.00013"/>
 		<axis xyz="1.0 0 0"/>
 		<limit effort="5.428" lower="-2.08567" upper="2.08567" velocity="7.33998"/>
